File: hardware/bmp180_tryout.kicad_pcb (KiCad board)
At the start: 2 copper layers, 4 parts, among them J1 BMP180_HEADER, U1 BMP180

Commit message: update,
Other:
- board outline added: 11.9 x 9.9 mm
- net class Default removed
